File: board templates/large/template_L_01.sch (EAGLE design)
At the start: 2 parts

Commit message: board templates SML
Other:
- note added: "large template"
- note removed: "template"
Changed lines of the file:
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@@
 <sheet>
 <plain>
-<text x="132.08" y="170.18" size="4.318" layer="94" font="vector">template</text>
+<text x="132.08" y="170.18" size="4.318" layer="94" font="vector">large template</text>
 </plain>
 <instances>
