File: board templates/medium/template_M_01.brd (EAGLE design)
At the start: 29.7 x 47.5 mm, 2 parts

Commit message: board templates SML
Parts:
- moved U$1 10.8 mm to (54.0, 22.9)
- moved U$2 0.52 mm to (4.45, 22.9)
Other:
- board size 29.7 x 47.5 mm -> 40.6 x 45.7 mm
Changed lines of the file:
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@@
 <setting verticaltext="up"/>
 </settings>
-<grid distance="0.01" unitdist="inch" unit="inch" style="dots" multiple="1" display="yes" altdistance="0.01" altunitdist="mm" altunit="mm"/>
+<grid distance="0.025" unitdist="inch" unit="inch" style="dots" multiple="1" display="yes" altdistance="0.01" altunitdist="mm" altunit="mm"/>
 <layers>
 <layer number="1" name="Top" color="4" fill="1" visible="yes" active="yes"/>
@@
 <board>
 <plain>
-<wire x1="13.335" y1="47.498" x2="34.163" y2="47.498" width="0" layer="20"/>
-<wire x1="34.163" y1="47.498" x2="38.608" y2="43.053" width="0" layer="20" curve="-90"/>
-<wire x1="13.335" y1="47.498" x2="8.89" y2="43.053" width="0" layer="20" curve="90"/>
-<wire x1="8.89" y1="43.053" x2="8.89" y2="41.148" width="0" layer="20"/>
-<wire x1="38.608" y1="43.053" x2="38.608" y2="41.148" width="0" layer="20"/>
-<wire x1="34.163" y1="0" x2="13.335" y2="0" width="0" layer="20"/>
+<wire x1="13.335" y1="45.72" x2="45.085" y2="45.72" width="0" layer="20"/>
+<wire x1="45.085" y1="45.72" x2="49.53" y2="41.275" width="0" layer="20" curve="-90"/>
+<wire x1="49.53" y1="41.275" x2="49.53" y2="40.64" width="0" layer="20"/>
+<wire x1="13.335" y1="45.72" x2="8.89" y2="41.275" width="0" layer="20" curve="90"/>
+<wire x1="8.89" y1="41.275" x2="8.89" y2="40.64" width="0" layer="20"/>
+<wire x1="13.335" y1="0" x2="45.085" y2="0" width="0" layer="20"/>
+<wire x1="45.085" y1="0" x2="49.53" y2="4.445" width="0" layer="20" curve="90"/>
+<wire x1="49.53" y1="4.445" x2="49.53" y2="5.08" width="0" layer="20"/>
 <wire x1="13.335" y1="0" x2="8.89" y2="4.445" width="0" layer="20" curve="-90"/>
-<wire x1="34.163" y1="0" x2="38.608" y2="4.445" width="0" layer="20" curve="90"/>
-<wire x1="38.608" y1="4.445" x2="38.608" y2="5.588" width="0" layer="20"/>
-<wire x1="8.89" y1="4.445" x2="8.89" y2="5.588" width="0" layer="20"/>
+<wire x1="8.89" y1="4.445" x2="8.89" y2="5.08" width="0" layer="20"/>
 </plain>
 <attributes>
@@
 </autorouter>
 <elements>
-<element name="U$1" library="mentor2" package="OTHERSNAP-OUT" value="OTHERSNAP-OUT" x="43.18" y="23.368"/>
-<element name="U$2" library="mentor2" package="OTHERSNAP-IN" value="OTHERSNAP-IN" x="4.318" y="23.368"/>
+<element name="U$1" library="mentor2" package="OTHERSNAP-OUT" value="OTHERSNAP-OUT" x="53.975" y="22.86"/>
+<element name="U$2" library="mentor2" package="OTHERSNAP-IN" value="OTHERSNAP-IN" x="4.445" y="22.86"/>
 </elements>
 <signals>
@@
 <contactref element="U$1" pad="GND"/>
 <contactref element="U$2" pad="GND"/>
-<wire x1="4.318" y1="18.288" x2="43.18" y2="18.288" width="0" layer="19" extent="1-1"/>
+<wire x1="4.445" y1="17.78" x2="53.975" y2="17.78" width="0" layer="19" extent="1-1"/>
 </signal>
 <signal name="N$8">
@@
 <contactref element="U$2" pad="VCC"/>
 <contactref element="U$1" pad="VCC"/>
-<wire x1="4.318" y1="28.448" x2="43.18" y2="28.448" width="0" layer="19" extent="1-1"/>
+<wire x1="4.445" y1="27.94" x2="53.975" y2="27.94" width="0" layer="19" extent="1-1"/>
 </signal>
 </signals>
